Commit message: Working SLAM and map generation state

File: src/my_bot/urdf/my_bot.urdf (robot description, URDF)
Before this commit: robot delivery_bot, 6 links, 5 joints
Links:
- link caster_wheel: geometry collision sphere radius=0.03; visual sphere radius=0.03
Joints:
- joint base_joint: origin xyz=0 0 0.05 rpy=0 0 0 -> xyz=0 0 0 rpy=0 0 0
- joint caster_joint: origin xyz=-0.15 0 -0.02 -> xyz=-0.15 0 -0.03
- joint left_wheel_joint: axis 0 1 0 -> 0 0 1; origin xyz=0 0.20 -0.02 rpy=0 0 0 -> xyz=0 0.15 0.07 rpy=0 0 0
- joint lidar_joint: origin xyz=0 0 0.1 rpy=0 0 0 -> xyz=0 0 0.15 rpy=0 0 0
- joint right_wheel_joint: axis 0 1 0 -> 0 0 1; origin xyz=0 -0.20 -0.02 rpy=0 0 0 -> xyz=0 -0.15 0.07 rpy=0 0 0

Commit message: Added RF2O odometry and updated robot navigation

File: src/my_bot/urdf/my_bot.urdf (robot description, URDF)
Before this commit: robot delivery_bot, 6 links, 5 joints
Joints:
- joint left_wheel_joint: axis 0 0 1 -> 0 1 0; origin xyz=0 0.15 0.07 rpy=0 0 0 -> xyz=0 0.18 0 rpy=0 0 0
- joint right_wheel_joint: axis 0 0 1 -> 0 -1 0; origin xyz=0 -0.15 0.07 rpy=0 0 0 -> xyz=0 -0.18 0 rpy=0 0 0
